File: PROpendousX/Hardware/PROpendousX/PROpendousX-DDR3.sch (KiCad schematic (older format))
At the start: 6 parts

Commit message: Progress update to PROpendousX design.
Parts:
- added R?: 240, symbol R_MINI
- added R? (x4): 0, symbol R_MINI_ARRAY4
- added R?: 47, symbol R_MINI_ARRAY4
- IC?: value AM335X_ZCZ -> AM335X
Connections:
- wire segments 9 -> 55
- no-connect marks 0 -> 5
Other:
- note added: "1%"
- note added: "Notes:\n - Errata 3.1.2 Take note of Self-Refresh issue\n - Signal terminators are required for the CK and ADDR_CTRL net classes while DATA class uses ODT\n - Termination resistors should be able to dissipate Power=(13mA^2)*47ohm=8mW\n - If using resistor packs for termination, isolate data/ctrl/addr groups\n - per Micron Note TN-00-06 use low inductance and low ESR caps around DDR IC\n - place b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"
- note removed: "Notes:\n - per Micron Note TN-00-06 use low inductance and low ESR caps around DDR IC\n - place bypass caps near each signal via for power plane stitching"
