File: PROpendousX/Hardware/PROpendousX/PROpendousX-Ethernet.sch (KiCad schematic (older format))
At the start: 10 parts

Commit message: Progress update to PROpendousX design.
Parts:
- removed U? (x2): JG0-0024NL, symbol ETH_JACK_DUAL_JG0-002XNL
- added U?: JK0-0133NL, symbol ETH_JACK_JK0-0133NL
- added U?: L829-1J1T-43, symbol ETH_JACK_L829-1J1T-43
- IC?: value AM335X_ZCZ -> AM335X
Connections:
- net labels added: POE_CT_VN, POE_CT_VP, SPI1_CS0, SPI1_MISO, SPI1_MOSI, SPI1_SCLK
- wire segments 21 -> 25
Other:
- note added: "Used in\nLCD Sheet"
- moved on the sheet: IC?I, R?
