File: PROpendousX/Hardware/PROpendousX/PROpendousX-LCD.sch (KiCad schematic (older format))
At the start: 16 parts

Commit message: Progress update to PROpendousX design.
Parts:
- removed C?: 0u1, symbol C_MINI
- removed IC?: CAT4237, symbol BOOST_DC-DC_SOT23-5
- removed R?: 0, symbol R_MINI
- added IC?: TB62737FUG, symbol TB62737FUG_LED_BOOST
- added IC?: MCP47x6, symbol MCP47X6_DAC
- added IC?: AM335X, symbol AM335X_ZCZ
- added L? (x2): FB, symbol L_MINI
- added R? (x3): 47k, symbol R_MINI
- added R? (x2): 16k, symbol R_MINI
- added R?: 100, symbol R_MINI
- C?: value 4u7 -> 2u2
- IC?: value AM335X_ZCZ -> AM335X
- L?: value 33uH -> 4.7uH
- R?: value 47k -> 82k
- R?: value 15 -> 16
Connections:
- net labels added: AIN0-XPUL, AIN1-XNNSW-XNUR, AIN2-YPNSW-VPLL, AIN3-YNNSW-VNLR, AIN4-WPNSW, GNDSHIELD, GND_BOOST, SPI1_CS0, SPI1_MOSI, SPI1_SCLK, VDD_3V3, VDD_BOOST
- net labels removed: GPMC_ADVn_ALE
- wire segments 36 -> 55
Other:
- note added: "2.5V"
- note added: "MCP47x6A0 has I2C address 1100000b = 0x60 = 96"
- note added: "Notes:\n - Errata 3.1.1 LCD pins have reverse color assignment in RGB888 mode:\n LCD_Data[23..0] = B[0]G[0]R[0]B[1]G[1]R[1]B[2]R[2]B[7:3]G[7:2]R[7:3]\n - LCD_AC_BIAS_EN is Data Valid signal"
- note added: "Using a DAC ensures no\naudible noise is produced"
- note removed: "1%"
- moved on the sheet: C?, IC?H, L?, R?, U?
