File: PROpendousX/Hardware/PROpendousX/PROpendousX-Opennect_Connector.sch (KiCad schematic (older format))
At the start: 19 parts

Commit message: Progress update to PROpendousX design.
Parts:
- removed C? (x4): 4u7, symbol C_MINI
- removed D?: MBR120, symbol D_SCHOTTKY
- removed IC? (x2): AP7361, symbol AP7361_DFN
- removed J?: DC_IN, symbol DC_POWER_JACK
- removed R? (x2): 249k, symbol R_MINI
- removed R? (x2): 47k, symbol R_MINI
- added IC? (x3): AM335X, symbol AM335X_ZCZ
- C?: value 0u1 -> 1u0
- IC?: value AM335X_ZCZ -> AM335X
Connections:
- net labels added: CLKOUT1, I2C0_SCL, I2C0_SDA, LCD_AC_BIAS_EN, LCD_DATA0-GPMC_A0-SYS_BOOT0, LCD_DATA1-GPMC_A1-SYS_BOOT1, LCD_DATA10-GPMC_A14-SYS_BOOT10, LCD_DATA11-GPMC_A15-SYS_BOOT11, LCD_DATA12-GPMC_A16-SYS_BOOT12, LCD_DATA13-GPMC_A17-SYS_BOOT13, LCD_DATA14-GPMC_A18-SYS_BOOT14, LCD_DATA15-GPMC_A19-SYS_BOOT15, LCD_DATA2-GPMC_A2-SYS_BOOT2, LCD_DATA3-GPMC_A3-SYS_BOOT3, LCD_DATA4-GPMC_A4-SYS_BOOT4, LCD_DATA5-GPMC_A5-SYS_BOOT5, LCD_DATA6-GPMC_A6-SYS_BOOT6, LCD_DATA7-GPMC_A7-SYS_BOOT7, LCD_DATA8-GPMC_A12-SYS_BOOT8, LCD_DATA9-GPMC_A13-SYS_BOOT9, LCD_HSYNC, LCD_PCLK, LCD_VSYNC, SPI0_CS0, SPI0_CS1, SPI0_MISO, SPI0_MOSI, SPI0_SCLK, UART0_CTSn, UART0_RTSn, UART0_RXD, UART0_TXD, VDDIO
- net labels removed: VDD3V3, VDDIO_3V3
- wire segments 105 -> 60
- no-connect marks 6 -> 0
Other:
- note removed: "10<ESR(mOhm)<300"
- note removed: "Full compatibility with the Opennect Specification\nrequires running the system from DC Power.\nD4 enables system 3V3 rail to partially power Opennect\nConnector when running off Li-Ion or USB to allow use\nof Opennect Modules that only require 3.3V rail."
- moved on the sheet: C?
