File: PROpendousX/Hardware/PROpendousX/PROpendousX-Power_Supply.sch (KiCad schematic (older format))
At the start: 12 parts

Commit message: Progress update to PROpendousX design.
Parts:
- removed BT?: BATTERY_LI-ION, symbol BATTERY_LI-ION
- removed IC?: LTC3576, symbol LTC3576
- removed Q?: MOSFET_N_OPENDOUS, symbol MOSFET_N_OPENDOUS
- added L?: FB, symbol L_MINI
- added TP1: VDD_MPU_MON, symbol CONN_1
- IC?: value AM335X_ZCZ -> AM335X
Connections:
- net labels added: VBB_MPU, VDDIO, VDD_3V3, VDD_CORE, VDD_MPU, VDD_PLL, VDD_RTC, VDD_SRAM_CORE, VDD_SRAM_MPU
- wire segments 20 -> 44
Other:
- note added: "TP1 = MPU_MON TP - Datasheet Figure 3-2"
- moved on the sheet: C?, IC?C, L?
