File: PROpendousX/Hardware/PROpendousX/PROpendousX-System.sch (KiCad schematic (older format))
At the start: 7 parts

Commit message: Progress update to PROpendousX design.
Parts:
- added C?: 0u1, symbol C_MINI
- added R? (x16): DNI, symbol R_MINI
- added R?: 10k, symbol R_MINI
- added R? (x16): 100k, symbol R_MINI
- added TP2: TESTOUT, symbol CONN_1
- added U?: JTAG, symbol CONN_CORTEX_DEBUG
- IC?: value AM335X_ZCZ -> AM335X
- X?: value 12MHz -> 24MHz
Connections:
- net labels added: CLKOUT1, LCD_DATA0-GPMC_A0-SYS_BOOT0, LCD_DATA1-GPMC_A1-SYS_BOOT1, LCD_DATA10-GPMC_A14-SYS_BOOT10, LCD_DATA11-GPMC_A15-SYS_BOOT11, LCD_DATA12-GPMC_A16-SYS_BOOT12, LCD_DATA13-GPMC_A17-SYS_BOOT13, LCD_DATA14-GPMC_A18-SYS_BOOT14, LCD_DATA15-GPMC_A19-SYS_BOOT15, LCD_DATA2-GPMC_A2-SYS_BOOT2, LCD_DATA3-GPMC_A3-SYS_BOOT3, LCD_DATA4-GPMC_A4-SYS_BOOT4, LCD_DATA5-GPMC_A5-SYS_BOOT5, LCD_DATA6-GPMC_A6-SYS_BOOT6, LCD_DATA7-GPMC_A7-SYS_BOOT7, LCD_DATA8-GPMC_A12-SYS_BOOT8, LCD_DATA9-GPMC_A13-SYS_BOOT9, PMIC_POWER_EN, TCK, TDI, TDO, TMS, VDDIO, ~TRSTn~
- wire segments 10 -> 536
Other:
- note added: "Boot Mode"
- note added: "RTC_KALDO_ENn LOW enables CAP_VDD_RTC\nto be sourced from an internal LDO"
- note added: "Table 26-5 of the AM335x TRM\nSYSBOOT[15:14] = 01b = 24MHz Crystal\nSYSBOOT[13:12] = 00b = Fixed\nSYSBOOT[11:6] = 000000b = Don't Care\nSYSBOOT[5] = 1b = CLKOUT1 Enabled\nSYSBOOT[4:0] = 11000b = SPI0..MMC0..USB0..UART0 Order"
