File: PROpendousX/Hardware/PROpendousX/PROpendousX-USB.sch (KiCad schematic (older format))
At the start: 1 part

Commit message: Progress update to PROpendousX design.
Parts:
- added IC?: AM335X, symbol AM335X_ZCZ
- added U?: PCIe-Mini, symbol PCIE_MINICARD
- IC?: value AM335X_ZCZ -> AM335X
Connections:
- new net I2C1_SCL: IC?.D15 (UART1_TXD-MMC2_SDWP-DCAN1_RX-I2C1_SCL-PR1_UART0_TXD-PR1_PRU0_PRU_R31_16-GPIO0_15)
- new net I2C1_SDA: IC?.D16 (UART1_RXD-MMC1_SDWP-DCAN1_TX-I2C1_SDA-PR1_UART0_RXD-PR1_PRU1_PRU_R31_16-GPIO0_14)
- new net I2C2_SCL: IC?.D17 (UART1_RTSn-TIMER5-DCAN0_RX-I2C2_SCL-SPI1_CS1-PR1_UART0_RTS_n-PR1_EDC_LATCH1_IN-GPIO0_13)
- new net I2C2_SDA: IC?.D18 (UART1_CTSn-TIMER6-DCAN0_TX-I2C2_SDA-SPI1_CS0-PR1_UART0_CTS_n-PR1_EDC_LATCH0_IN-GPIO0_12)
- no-connect marks 0 -> 6
Other:
- moved on the sheet: IC?K
Changed lines of the file:
@@
-EESchema Schematic File Version 2  date 12/9/2011 12:11:08 AM
+EESchema Schematic File Version 2  date 12/10/2011 4:37:07 AM
 LIBS:power
 LIBS:device
@@
 $Descr A4 11700 8267
 encoding utf-8
-Sheet 4 11
+Sheet 5 12
 Title "PROpendousX AM335x"
-Date "9 dec 2011"
+Date "10 dec 2011"
 Rev "1.0"
 Comp "Opendous Inc. (www.opendous.org)"
@@
 Comment4 "www.PROpendousX.org"
 $EndDescr
+Text GLabel 5800 6800 2    40   Input ~ 0
+I2C2_SCL
+Text GLabel 5800 6900 2    40   Input ~ 0
+I2C2_SDA
+Text GLabel 5800 6700 2    40   Input ~ 0
+I2C1_SDA
+Text GLabel 5800 6600 2    40   Input ~ 0
+I2C1_SCL
+$Comp
+L AM335X_ZCZ IC?
+U 14 1 4EE31E47
+P 800 6750
+F 0 "IC?" V 750 7000 60  0000 C CNN
+F 1 "AM335X" V 750 6650 60  0000 C CNN
+	14   800  6750
+	1    0    0    -1
+$EndComp
+NoConn ~ 6800 4550
+NoConn ~ 6800 4450
+NoConn ~ 6800 4300
+NoConn ~ 6800 4200
+NoConn ~ 6800 4050
+NoConn ~ 6800 3950
+$Comp
+L GNDSHIELD #PWR?
+U 1 1 4EE30E08
+P 9000 1800
+F 0 "#PWR?" H 9000 1850 40  0001 C CNN
+F 1 "GNDSHIELD" H 9000 1740 25  0000 C CNN
+	1    9000 1800
+	1    0    0    -1
+$EndComp
+$Comp
+L PCIE_MINICARD U?
+U 1 1 4EE2ECE4
+P 5900 4700
+F 0 "U?" H 5900 4600 60  0000 C CNN
+F 1 "PCIe-Mini" H 5900 4800 60  0000 C CNN
+	1    5900 4700
+	1    0    0    -1
+$EndComp
 $Comp
 L AM335X_ZCZ IC?
 U 11 1 4EE13B6E
-P 3200 3050
-F 0 "IC?" V 3150 3350 60  0000 C CNN
-F 1 "AM335X_ZCZ" V 3150 2750 60  0000 C CNN
-	11   3200 3050
+P 5300 1750
+F 0 "IC?" V 5250 2050 60  0000 C CNN
+F 1 "AM335X" V 5250 1450 60  0000 C CNN
+	11   5300 1750
 	1    0    0    -1
 $EndComp
