File: PROpendousX/Hardware/PROpendousX/PROpendousX.sch (KiCad schematic (older format))
At the start: 0 parts

Commit message: Progress update to PROpendousX design.
Changed lines of the file:
@@
-EESchema Schematic File Version 2  date 12/9/2011 12:11:08 AM
+EESchema Schematic File Version 2  date 12/10/2011 4:37:07 AM
 LIBS:power
 LIBS:device
@@
 LIBS:contrib
 LIBS:valves
+LIBS:opendous
+LIBS:Opennect_Schematic_Symbols_Library
 LIBS:PROpendousX-cache
 EELAYER 25  0
@@
 $Descr A4 11700 8267
 encoding utf-8
-Sheet 1 11
+Sheet 1 12
 Title "PROpendousX AM335x"
-Date "9 dec 2011"
+Date "10 dec 2011"
 Rev "1.0"
 Comp "Opendous Inc. (www.opendous.org)"
@@
 $EndDescr
 $Sheet
-S 900  7200 3000 300
+S 900  3700 3000 300
+U 4EE28EE1
+F0 "Power_Manager" 60
+F1 "PROpendousX-Power_Manager.sch" 60
+$EndSheet
+$Sheet
+S 4500 4400 3000 300
 U 4EE13B4B
 F0 "Vias" 60
@@
 	4400 6100 4000 6100
 $Sheet
-S 900  5800 3000 300
+S 4500 3000 3000 300
 U 4EE13939
 F0 "Ethernet" 60
@@
 $EndSheet
 $Sheet
-S 900  6500 3000 300
+S 4500 3700 3000 300
 U 4EE138FD
 F0 "USB" 60
@@
 $EndSheet
 $Sheet
-S 900  5100 3000 300
+S 4500 2300 3000 300
 U 4EE13170
 F0 "MMC" 60
@@
 $EndSheet
 $Sheet
-S 900  4400 3000 300
+S 4500 900  3000 300
 U 4EE124E1
 F0 "Signal_MUX" 60
@@
 	4000 6500 4000 6100
 $Sheet
-S 900  3700 3000 300
+S 4500 1600 3000 300
 U 4EDEB54F
 F0 "LCD" 60
